File: 2s3pShortArraySV4/solar-panel-side-Z.kicad_pcb (KiCad board)
At the start: 4 copper layers, 100 x 100 mm, 15 parts, among them J1 2053380005-CONNECTOR, U1 APDS9960_Breakout, U2 DRV2605L_Breakout, U3 MCP9808_Breakout, U4 BNO080_Breakout, U5 MCP9601_Breakout

Commit message: Add files via upload
Parts:
- moved U2 1.88 mm to (138.2, 69.2)
- moved U1 0.36 mm to (160.6, 110.3)
- moved U3 0.22 mm to (137.0, 79.5)
- moved D1 0.14 mm to (120.0, 85.5)
Routing:
- net Net-(U2-Pad6): track 9000.5 -> 8998.4 mm
- net SCL: track 100.2 -> 101.8 mm
- net SDA: track 92.4 -> 93.9 mm
- net +3V3: track 117.7 -> 118.9 mm

Commit message: Add files via upload
Parts:
- J1: value 2053380005-CONNECTOR -> CON-5040500591; footprint SolarPanelBoards:CON_2053380005 -> SolarPanelBoards:CON_5040500591
- moved U5 63.3 mm to (171.2, 79.0)
- moved U4 0.75 mm to (148.0, 85.5)
- moved J1 0.50 mm to (141.8, 99.8)
Routing:
- net Net-(SC3-Pad2): track 82.3 -> 98.7 mm
- net +3V3: track 118.9 -> 135.1 mm, vias 2 -> 4
- net SDA: track 93.9 -> 105.3 mm, vias 2 -> 3
- net SCL: track 101.8 -> 113.1 mm, vias 2 -> 3
- net GND: track 44.6 -> 53.5 mm
- net VSOLAR: track 70.5 -> 70.0 mm
Other:
- outline, holes or cut-outs redrawn

Commit message: Add files via upload
Parts:
- moved U5 43.6 mm to (128.0, 73.2), turned to 90 degrees
- moved SC4 30.5 mm to (164.5, 106.2)
- moved SC3 30.3 mm to (134.5, 64.0)
- moved D2 28.8 mm to (135.0, 85.5), turned to 0 degrees
- moved U3 24.6 mm to (161.0, 74.0)
- moved U1 22.1 mm to (138.5, 111.5)
- moved U2 21.9 mm to (159.7, 64.5)
- moved U4 3.00 mm to (151.0, 85.5)
Routing:
- net GND: track 53.5 -> 19.5 mm
- net +3V3: track 135.1 -> 101.7 mm, vias 4 -> 3
- net SDA: track 105.3 -> 111.1 mm
- net Net-(SC3-Pad2): track 98.7 -> 94.0 mm
- net SCL: track 113.1 -> 109.6 mm
- net Net-(D2-Pad2): track 35.4 -> 37.4 mm
- net Net-(U2-Pad6): track 8998.4 -> 8997.3 mm
- net VSOLAR: track 70.0 -> 70.7 mm
Other:
- outline, holes or cut-outs redrawn
