File: 2s3pShortArraySV4/solar-panel-side+XY.kicad_pcb (KiCad board)
At the start: 4 copper layers, 83 x 98 mm, 13 parts, among them J1 2053380005-CONNECTOR, U1 APDS9960_Breakout, U2 BNO080_Breakout, U3 MCP9808_Breakout

Commit message: Add files via upload
Parts:
- moved D1 1.25 mm to (125.5, 91.0)
- moved U2 1.00 mm to (141.5, 96.8)
- moved U3 0.35 mm to (141.2, 116.2)
- moved D3 0.25 mm to (157.8, 92.0)
- moved J1 0.25 mm to (116.0, 109.5)
- moved SC2 0.25 mm to (117.0, 129.2)
- moved SC3 0.25 mm to (166.0, 129.2)
- moved U1 0.25 mm to (141.5, 133.0)
Routing:
- net Net-(SC5-Pad2): track 65.4 -> 70.2 mm
- net Net-(D1-Pad2): track 28.3 -> 26.3 mm
Other:
- outline, holes or cut-outs redrawn

Commit message: Add files via upload
Parts:
- J1: value 2053380005-CONNECTOR -> CON-5040500591; footprint SolarPanelBoards:CON_2053380005 -> SolarPanelBoards:CON_5040500591
- moved J1 1.03 mm to (116.9, 109.0)
Routing:
- net +3V3: track 91.4 -> 93.9 mm
- net VSOLAR: track 64.7 -> 64.1 mm
- net SDA: track 67.6 -> 68.2 mm
- net SCL: track 75.8 -> 76.3 mm

Commit message: Add files via upload
Other:
- rule trace_min: 0.2 -> 0.25
- rule via_min_size: 0.4 -> 0.8

Commit message: Add files via upload
Other:
- copper layers 4 -> 2
