File: 2s3pShortArraySV4/solar-panel-side-XY.kicad_pcb (KiCad board)
At the start: 4 copper layers, 83 x 98 mm, 13 parts, among them J1 2053380005-CONNECTOR, U1 APDS9960_Breakout, U2 DRV2605L_Breakout, U3 MCP9808_Breakout

Commit message: Add files via upload
Parts:
- moved U3 6.48 mm to (121.2, 114.9)
- moved U2 1.79 mm to (170.0, 106.8)
- moved U1 0.56 mm to (145.8, 111.2)
- moved D1 0.35 mm to (139.0, 125.2)
- moved J1 0.28 mm to (122.4, 125.5)
- moved D2 0.25 mm to (149.5, 125.2)
- moved D3 0.25 mm to (158.8, 125.2)
- moved SC4 0.25 mm to (144.8, 83.8)
- moved SC6 0.25 mm to (167.8, 83.8)
Routing:
- net SDA: track 71.7 -> 76.6 mm
- net SCL: track 75.1 -> 79.9 mm
- net GND: track 20.6 -> 24.3 mm
- net +3V3: track 84.8 -> 88.4 mm
- net Net-(U2-Pad6): track 9247.2 -> 9244.0 mm
- net VSOLAR: track 40.9 -> 41.6 mm
Other:
- outline, holes or cut-outs redrawn

Commit message: Add files via upload
Parts:
- J1: value 2053380005-CONNECTOR -> CON-5040500591; footprint SolarPanelBoards:CON_2053380005 -> SolarPanelBoards:CON_5040500591
- moved J1 1.37 mm to (123.5, 124.8)
Routing:
- net SDA: track 76.6 -> 68.1 mm
- net SCL: track 79.9 -> 72.9 mm
- net +3V3: track 88.4 -> 82.9 mm

Commit message: Add files via upload
Other:
- rule trace_min: 0.2 -> 0.25
- rule via_min_size: 0.4 -> 0.8
