File: Yearling 2 Solar Update 2.0/solar-panel-side-Z.kicad_sch (KiCad schematic)
At the start: 35 parts, among them IC1 VEML7700, J1 CON-5040500591, J2 Screw_Terminal_01x02, J3 Conn_01x01, J4 Conn_01x01, J5 Conn_01x01, J6 Conn_01x01, U2 DRV2605LDGS, U3 MCP9808_DFN, U4 MCP96L01T-E_MX

Commit message: Boards as Ordered Jan 31,2023
Connections:
- net +3V3: now also U3.6 (A1), U3.7 (A0)
- net GND: no longer U3.6 (A1), U3.7 (A0)
Changed lines of the file:
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@@
   (junction (at 109.22 88.9) (diameter 0) (color 0 0 0 0)
   )
+  (junction (at 32.512 96.266) (diameter 0) (color 0 0 0 0)
+  )
   (junction (at 137.16 77.47) (diameter 0) (color 0 0 0 0)
   )
@@
   (junction (at 97.79 96.52) (diameter 0) (color 0 0 0 0)
   )
-  (junction (at 33.02 100.33) (diameter 0) (color 0 0 0 0)
-  )
   (junction (at 44.45 137.16) (diameter 0) (color 0 0 0 0)
   )
@@
   (junction (at 134.62 77.47) (diameter 0) (color 0 0 0 0)
   )
+  (junction (at 45.72 76.962) (diameter 0) (color 0 0 0 0)
+  )
   (junction (at 116.84 99.06) (diameter 0) (color 0 0 0 0)
   )
@@
   )
   (junction (at 107.95 120.65) (diameter 0) (color 0 0 0 0)
-  )
-  (junction (at 33.02 97.79) (diameter 0) (color 0 0 0 0)
   )
   (no_connect (at 137.16 105.41))
@@
     (stroke (width 0) (type default) (color 0 0 0 0))
   )
-  (wire (pts (xy 33.02 95.25) (xy 33.02 97.79))
+  (wire (pts (xy 32.512 95.504) (xy 35.56 95.504))
     (stroke (width 0) (type default) (color 0 0 0 0))
   )
@@
     (stroke (width 0) (type default) (color 0 0 0 0))
   )
-  (wire (pts (xy 45.72 76.2) (xy 45.72 80.01))
+  (wire (pts (xy 45.72 76.2) (xy 45.72 76.962))
     (stroke (width 0) (type default) (color 0 0 0 0))
   )
@@
     (stroke (width 0) (type default) (color 0 0 0 0))
   )
+  (wire (pts (xy 17.526 76.962) (xy 17.526 96.266))
+    (stroke (width 0) (type default) (color 0 0 0 0))
+  )
   (wire (pts (xy 139.7 77.47) (xy 139.7 81.28))
     (stroke (width 0) (type default) (color 0 0 0 0))
@@
     (stroke (width 0) (type default) (color 0 0 0 0))
   )
-  (wire (pts (xy 33.02 97.79) (xy 33.02 100.33))
+  (wire (pts (xy 45.72 76.962) (xy 17.526 76.962))
     (stroke (width 0) (type default) (color 0 0 0 0))
   )
@@
     (stroke (width 0) (type default) (color 0 0 0 0))
   )
+  (wire (pts (xy 32.512 96.266) (xy 32.512 95.504))
+    (stroke (width 0) (type default) (color 0 0 0 0))
+  )
   (wire (pts (xy 57.15 151.13) (xy 62.23 151.13))
     (stroke (width 0) (type default) (color 0 0 0 0))
@@
     (stroke (width 0) (type default) (color 0 0 0 0))
   )
+  (wire (pts (xy 35.56 97.79) (xy 32.512 97.79))
+    (stroke (width 0) (type default) (color 0 0 0 0))
+  )
   (wire (pts (xy 106.68 110.49) (xy 107.95 110.49))
     (stroke (width 0) (type default) (color 0 0 0 0))
@@
     (stroke (width 0) (type default) (color 0 0 0 0))
   )
+  (wire (pts (xy 45.72 76.962) (xy 45.72 80.01))
+    (stroke (width 0) (type default) (color 0 0 0 0))
+  )
   (wire (pts (xy 25.4 146.05) (xy 31.75 146.05))
     (stroke (width 0) (type default) (color 0 0 0 0))
@@
     (stroke (width 0) (type default) (color 0 0 0 0))
   )
+  (wire (pts (xy 17.526 96.266) (xy 32.512 96.266))
+    (stroke (width 0) (type default) (color 0 0 0 0))
+  )
   (wire (pts (xy 64.77 158.75) (xy 67.31 158.75))
     (stroke (width 0) (type default) (color 0 0 0 0))
@@
     (stroke (width 0) (type default) (color 0 0 0 0))
   )
-  (wire (pts (xy 35.56 97.79) (xy 33.02 97.79))
-    (stroke (width 0) (type default) (color 0 0 0 0))
-  )
   (wire (pts (xy 198.12 88.9) (xy 198.12 82.55))
     (stroke (width 0) (type default) (color 0 0 0 0))
@@
     (stroke (width 0) (type default) (color 0 0 0 0))
   )
+  (wire (pts (xy 35.56 95.504) (xy 35.56 95.25))
+    (stroke (width 0) (type default) (color 0 0 0 0))
+  )
   (wire (pts (xy 179.07 49.53) (xy 201.93 49.53))
     (stroke (width 0) (type default) (color 0 0 0 0))
@@
     (stroke (width 0) (type default) (color 0 0 0 0))
   )
+  (wire (pts (xy 32.512 97.79) (xy 32.512 96.266))
+    (stroke (width 0) (type default) (color 0 0 0 0))
+  )
   (wire (pts (xy 67.31 158.75) (xy 67.31 165.1))
     (stroke (width 0) (type default) (color 0 0 0 0))
@@
     (stroke (width 0) (type default) (color 0 0 0 0))
   )
-  (wire (pts (xy 35.56 95.25) (xy 33.02 95.25))
-    (stroke (width 0) (type default) (color 0 0 0 0))
-  )
