File: Yearling 2 Solar Update 2.0/no cutout/solar-panel-NoCutout.kicad_pcb (KiCad board)
At the start: 4 copper layers, 83 x 98 mm, 25 parts, among them IC1 VEML7700, J1 CON-5040500591, J2 Conn_01x01, J3 Conn_01x01, J4 Conn_01x01, J5 Conn_01x01, U2 MCP9808_DFN, U3 DRV2605LDGS

Commit message: Boards as Ordered Jan 31,2023
Routing:
- net GND: track 47.1 -> 44.8 mm
Changed lines of the file:
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@@
   (segment (start 144.45 161.94) (end 144.45 156.25) (width 0.5) (layer "F.Cu") (net 1))
   (segment (start 154.45 114.42) (end 153.7 113.67) (width 0.25) (layer "F.Cu") (net 1))
-  (segment (start 149.3 119.34) (end 151.25 119.34) (width 0.25) (layer "F.Cu") (net 1))
   (segment (start 160.9 114.35) (end 160.75 114.5) (width 0.25) (layer "F.Cu") (net 1))
   (segment (start 160.57 109.96) (end 163.89 109.96) (width 0.25) (layer "F.Cu") (net 1))
@@
   (segment (start 153.7 113.67) (end 153 113.67) (width 0.25) (layer "F.Cu") (net 1))
   (segment (start 160.4 114.85) (end 160.75 114.5) (width 0.25) (layer "F.Cu") (net 1))
-  (segment (start 151.25 119.34) (end 151.53 119.62) (width 0.25) (layer "F.Cu") (net 1))
   (segment (start 155.2 113.67) (end 154.485 114.385) (width 0.25) (layer "F.Cu") (net 1))
   (segment (start 148.885 112.89) (end 149.675 112.1) (width 0.25) (layer "F.Cu") (net 1))
